Commit message: add something related to moveit

File: robotis_manipulator_h_description/urdf/robotis_manipulator_h.xacro (robot description, xacro)
@@ -275,8 +275,14 @@
   <!-- End Effector -->
   <link name="end_effector">
-    <visual>
+    <collision>
       <origin xyz="0.0 0.0 0.0" rpy="0 0 0" />
       <geometry>
-        <box size="0.005 0.005 0.005" />
+        <cylinder length="0.01" radius="0.01"/>
+      </geometry>
+    </collision>
+    <visual>
+      <origin xyz="0.0 0.0 0.0" rpy="0 0 0" />
+      <geometry>
+        <cylinder length="0.01" radius="0.01"/>
       </geometry>
       <material name="red"/>
